File: PCB/CTL_KiCad/CTL.sch (KiCad schematic (older format))
At the start: 17 parts, among them J1_2 Conn_02x08_Counter_Clockwise, J3 Conn_01x10, J4 SW_DIP_x01, Q1 Q_NPN_EBC, SW1 Rotary_Encoder_Switch

Commit message: Initial Version of KiCAD based CTL board.
Parts:
- Q1: DigiKey (none) -> 2N4401BU
- R1, R2, R3, R4, R5: footprint Resistor_THT:R_Axial_DIN0204_L3.6mm_D1.6mm_P5.08mm_Vertical -> Resistor_THT:R_Axial_DIN0204_L3.6mm_D1.6mm_P5.08mm_Horizontal
- SG1: value Buzzer -> CEM-1201(50); footprint (none) -> FDL3_KiCad:CEM-1201(50); DigiKey (none) -> 102-1152-ND
- SW1: footprint Rotary_Encoder:RotaryEncoder_Alps_EC11E-Switch_Vertical_H20mm -> FDL3_KiCad:PEC11R-4215K-S0024
Changed lines of the file:
@@
 F 0 "SW1" H 5200 3733 50  0000 C CNN
 F 1 "Rotary_Encoder_Switch" H 5200 3824 50  0000 C CNN
-F 2 "Rotary_Encoder:RotaryEncoder_Alps_EC11E-Switch_Vertical_H20mm" H 5050 4260 50  0001 C CNN
+F 2 "FDL3_KiCad:PEC11R-4215K-S0024" H 5050 4260 50  0001 C CNN
 F 3 "~" H 5200 4360 50  0001 C CNN
 	1    5200 4100
@@
 F 0 "R1" H 4770 2096 50  0000 L CNN
 F 1 "1k" H 4770 2005 50  0000 L CNN
-F 2 "Resistor_THT:R_Axial_DIN0204_L3.6mm_D1.6mm_P5.08mm_Vertical" V 4630 2050 50  0001 C CNN
+F 2 "Resistor_THT:R_Axial_DIN0204_L3.6mm_D1.6mm_P5.08mm_Horizontal" V 4630 2050 50  0001 C CNN
 F 3 "~" H 4700 2050 50  0001 C CNN
 	1    4700 2050
@@
 F 0 "R2" H 4770 2896 50  0000 L CNN
 F 1 "1k" H 4770 2805 50  0000 L CNN
-F 2 "Resistor_THT:R_Axial_DIN0204_L3.6mm_D1.6mm_P5.08mm_Vertical" V 4630 2850 50  0001 C CNN
+F 2 "Resistor_THT:R_Axial_DIN0204_L3.6mm_D1.6mm_P5.08mm_Horizontal" V 4630 2850 50  0001 C CNN
 F 3 "~" H 4700 2850 50  0001 C CNN
 	1    4700 2850
@@
 F 0 "R3" H 4770 3696 50  0000 L CNN
 F 1 "1k" H 4770 3605 50  0000 L CNN
-F 2 "Resistor_THT:R_Axial_DIN0204_L3.6mm_D1.6mm_P5.08mm_Vertical" V 4630 3650 50  0001 C CNN
+F 2 "Resistor_THT:R_Axial_DIN0204_L3.6mm_D1.6mm_P5.08mm_Horizontal" V 4630 3650 50  0001 C CNN
 F 3 "~" H 4700 3650 50  0001 C CNN
 	1    4700 3650
@@
 F 0 "R4" H 4870 4496 50  0000 L CNN
 F 1 "4.7k" H 4870 4405 50  0000 L CNN
-F 2 "Resistor_THT:R_Axial_DIN0204_L3.6mm_D1.6mm_P5.08mm_Vertical" V 4730 4450 50  0001 C CNN
+F 2 "Resistor_THT:R_Axial_DIN0204_L3.6mm_D1.6mm_P5.08mm_Horizontal" V 4730 4450 50  0001 C CNN
 F 3 "~" H 4800 4450 50  0001 C CNN
 	1    4800 4450
@@
 F 0 "R5" H 6770 2296 50  0000 L CNN
 F 1 "1k" H 6770 2205 50  0000 L CNN
-F 2 "Resistor_THT:R_Axial_DIN0204_L3.6mm_D1.6mm_P5.08mm_Vertical" V 6630 2250 50  0001 C CNN
+F 2 "Resistor_THT:R_Axial_DIN0204_L3.6mm_D1.6mm_P5.08mm_Horizontal" V 6630 2250 50  0001 C CNN
 F 3 "~" H 6700 2250 50  0001 C CNN
 	1    6700 2250
@@
 F 2 "Package_TO_SOT_THT:TO-92" H 7200 2100 50  0001 C CNN
 F 3 "~" H 7000 2000 50  0001 C CNN
+F 4 "2N4401BU" H 7450 1850 50  0000 C CNN "DigiKey"
 	1    7000 2000
 	1    0    0    -1
@@
 P 7300 1600
 F 0 "SG1" H 7452 1629 50  0000 L CNN
-F 1 "Buzzer" H 7452 1538 50  0000 L CNN
-F 2 "" V 7275 1700 50  0001 C CNN
+F 1 "CEM-1201(50)" H 7452 1538 50  0000 L CNN
+F 2 "FDL3_KiCad:CEM-1201(50)" V 7275 1700 50  0001 C CNN
 F 3 "~" V 7275 1700 50  0001 C CNN
+F 4 "102-1152-ND" H 7300 1600 50  0001 C CNN "DigiKey"
 	1    7300 1600
 	1    0    0    -1
